File: Ver 2.1 Rel 0/Eagle PCB/Dual v12.sch (EAGLE design)
At the start: 137 parts, among them J1 DCJ0202PIN, J3 SCREW-TERM_5MM_BG, J4 22-23-2041, J5 22-23-2041, J6 SCREW-TERM_5MM_BG, J7 SCREW-TERM_5MM_BG, K1 G6N-2-Y, K2 G6N-2-Y, Q1 MMBT3906, Q2 Si2307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

Commit message: added BOM
Parts:
- C14: PARTNO STOCK: 1UF/10V 20% TDK -> DK: 311-1456-1-ND
- R11: PARTNO STOCK: 10R -> STOCK
- TP1, TP2, TP3, U$2, U$3: PARTNO (none) -> *
Changed lines of the file:
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@@
 </part>
 <part name="C14" library="ipc-7351-capacitor" deviceset="CAPACITOR_" device="0805N" value="1uF/25V">
-<attribute name="PARTNO" value="STOCK: 1UF/10V 20% TDK"/>
+<attribute name="PARTNO" value="DK: 311-1456-1-ND"/>
 </part>
 <part name="SUPPLY12" library="supply2" deviceset="GND" device=""/>
@@
 </part>
 <part name="R11" library="ipc-7351-resistor" deviceset="RESISTOR_" device="0603" value="100R">
-<attribute name="PARTNO" value="STOCK: 10R"/>
+<attribute name="PARTNO" value="STOCK"/>
 </part>
 <part name="SUPPLY66" library="Misc Voltages" deviceset="+3.3V" device=""/>
@@
 <attribute name="PARTNO" value="*"/>
 </part>
-<part name="TP1" library="testpad" deviceset="TPSQ" device="TP08R" value="TPSQTP08R"/>
-<part name="TP2" library="testpad" deviceset="TPSQ" device="TP14SQ" value="TPSQTP14SQ"/>
-<part name="TP3" library="testpad" deviceset="TPSQ" device="TP14SQ" value="TPSQTP14SQ"/>
+<part name="TP1" library="testpad" deviceset="TPSQ" device="TP08R" value="TPSQTP08R">
+<attribute name="PARTNO" value="*"/>
+</part>
+<part name="TP2" library="testpad" deviceset="TPSQ" device="TP14SQ" value="TPSQTP14SQ">
+<attribute name="PARTNO" value="*"/>
+</part>
+<part name="TP3" library="testpad" deviceset="TPSQ" device="TP14SQ" value="TPSQTP14SQ">
+<attribute name="PARTNO" value="*"/>
+</part>
 <part name="SUPPLY99" library="supply2" deviceset="GND" device=""/>
-<part name="U$2" library="Misc logo" deviceset="CC" device="NONE" value="CCNONE"/>
-<part name="U$3" library="Misc logo" deviceset="POLARITY" device=""/>
+<part name="U$2" library="Misc logo" deviceset="CC" device="NONE" value="CCNONE">
+<attribute name="PARTNO" value="*"/>
+</part>
+<part name="U$3" library="Misc logo" deviceset="POLARITY" device="">
+<attribute name="PARTNO" value="*"/>
+</part>
 </parts>
 <sheets>
@@
 <attribute name="PARTNO" x="281.94" y="2.54" size="1.778" layer="96" display="off"/>
 </instance>
-<instance part="TP1" gate="G$1" x="149.86" y="175.26" rot="R90"/>
-<instance part="TP2" gate="G$1" x="101.6" y="63.5" rot="R180"/>
-<instance part="TP3" gate="G$1" x="99.06" y="76.2" rot="R90"/>
+<instance part="TP1" gate="G$1" x="149.86" y="175.26" rot="R90">
+<attribute name="PARTNO" x="149.86" y="175.26" size="1.778" layer="96" display="off"/>
+</instance>
+<instance part="TP2" gate="G$1" x="101.6" y="63.5" rot="R180">
+<attribute name="PARTNO" x="101.6" y="63.5" size="1.778" layer="96" display="off"/>
+</instance>
+<instance part="TP3" gate="G$1" x="99.06" y="76.2" rot="R90">
+<attribute name="PARTNO" x="99.06" y="76.2" size="1.778" layer="96" display="off"/>
+</instance>
 <instance part="SUPPLY99" gate="GND" x="93.98" y="71.12"/>
-<instance part="U$3" gate="G$1" x="40.64" y="243.84"/>
+<instance part="U$3" gate="G$1" x="40.64" y="243.84">
+<attribute name="PARTNO" x="40.64" y="243.84" size="1.778" layer="96" display="off"/>
+</instance>
 </instances>
 <busses>
@@
 <instance part="U6" gate="B" x="160.02" y="203.2"/>
 <instance part="U6" gate="P" x="167.64" y="175.26"/>
-<instance part="U$2" gate="G$1" x="281.94" y="2.54"/>
+<instance part="U$2" gate="G$1" x="281.94" y="2.54">
+<attribute name="PARTNO" x="281.94" y="2.54" size="1.778" layer="96" display="off"/>
+</instance>
 </instances>
 <busses>
